Commit message: Add files via upload

File: 3Dvisualisation/robot_description/urdf/robot.xacro (robot description, xacro)
@@ -158,4 +158,19 @@
 	<xacro:default_inertial mass="0.01"/>
 </link>
+<link name="endeffector">
+	<visual name="end_visual">
+	<geometry>
+	<mesh filename="package://robot_description/meshes/end.stl"/>
+	</geometry>
+	<origin rpy= " 0 0 0" xyz ="0 0 0"/>
+	</visual>
+	<collision name="end_collision">
+	<geometry>
+	<mesh filename="package://robot_description/meshes/end.stl"/>
+	</geometry>
+	<origin rpy="0 0 0" xyz="0 0 0"/>
+	</collision>
+	<xacro:default_inertial mass="0.01"/>
+</link>
 <joint name="basetoworld" type="fixed">
 	<parent link="world"/>
@@ -172,5 +187,5 @@
 	<origin xyz ="0.14 0 -0.20"/>
 	<axis xyz = "0 0 1"/>
-	<limit effort="1000.0" lower="-1.0467" upper="1.0467" velocity="0.5"/>
+	<limit effort="1000.0" lower="-2.1" upper="2.1" velocity="0.5"/>
 </joint>
 <joint name="joint1" type="fixed">
@@ -185,5 +200,5 @@
 	<origin xyz ="0.14 0 -0.187"/>
 	<axis xyz = "0 0 1"/>
-	<limit effort="1000.0" lower="-1.0467" upper="1.0467" velocity="0.5"/>
+	<limit effort="1000.0" lower="-2.1" upper="2.1" velocity="0.5"/>
 </joint>
 <joint name="joint3" type ="fixed">
@@ -198,5 +213,5 @@
 	<origin xyz ="0.14 0 -0.187"/>
 	<axis xyz = "0 0 1"/>
-	<limit effort="1000.0" lower="-1.0467" upper="1.0467" velocity="0.5"/>
+	<limit effort="1000.0" lower="-2.1" upper="2.1" velocity="0.5"/>
 </joint>
 <joint name="joint5" type ="fixed">
@@ -211,5 +226,5 @@
 	<origin xyz ="0.14 0 -0.187"/>
 	<axis xyz = "0 0 1"/>
-	<limit effort="1000.0" lower="-1.0467" upper="1.0467" velocity="0.5"/>
+	<limit effort="1000.0" lower="-2.1" upper="2.1" velocity="0.5"/>
 </joint>
 <joint name="joint7" type ="fixed">
@@ -219,4 +234,11 @@
 	<limit effort="0" lower = "0.0" upper="0.0" velocity="0.0"/>
 </joint>
+<joint name="end" type="revolute">
+	<parent link="motor04"/>
+	<child link ="endeffector"/>
+	<origin xyz="0.12 -0.01 -0.185"/>
+	<axis xyz = "0 0 1"/>
+	<limit effort="1000.0" lower = "-2.1" upper="2.1" velocity="0.5"/>
+</joint>
 <transmission name="tran1">
     <type>transmission_interface/SimpleTransmission</type>
@@ -255,4 +277,14 @@
     </joint>
     <actuator name="motor4">
+      <hardwareInterface>hardware_interface/EffortJointInterface</hardwareInterface>
+      <mechanicalReduction>1</mechanicalReduction>
+    </actuator>
+  </transmission>
+<transmission name="tran4">
+    <type>transmission_interface/SimpleTransmission</type>
+    <joint name="end">
+      <hardwareInterface>hardware_interface/EffortJointInterface</hardwareInterface>
+    </joint>
+    <actuator name="motor5">
       <hardwareInterface>hardware_interface/EffortJointInterface</hardwareInterface>
       <mechanicalReduction>1</mechanicalReduction>
